Commit message: [update] URDF related and README

File: assets/h1_2/h1_2_simplified.urdf (robot description, URDF)
Before this commit: robot h1_5, 56 links, 55 joints
Links:
- link L_hand_base_link: geometry visual mesh filename=meshes/L_hand_base_link.STL
- link L_index_intermediate: geometry visual mesh filename=meshes/link16_L.STL
- link L_index_proximal: geometry visual mesh filename=meshes/link15_L.STL
- link L_middle_intermediate: geometry visual mesh filename=meshes/link18_L.STL
- link L_middle_proximal: geometry visual mesh filename=meshes/link17_L.STL
- link L_pinky_intermediate: geometry visual mesh filename=meshes/link22_L.STL
- link L_pinky_proximal: geometry visual mesh filename=meshes/link21_L.STL
- link L_ring_intermediate: geometry visual mesh filename=meshes/link20_L.STL
- link L_ring_proximal: geometry visual mesh filename=meshes/link19_L.STL
- link L_thumb_distal: geometry visual mesh filename=meshes/link14_L.STL
- link L_thumb_intermediate: geometry visual mesh filename=meshes/link13_L.STL
- link L_thumb_proximal: geometry visual mesh filename=meshes/link12_L.STL
- link L_thumb_proximal_base: geometry visual mesh filename=meshes/link11_L.STL
- link R_hand_base_link: geometry visual mesh filename=meshes/R_hand_base_link.STL
- link R_index_intermediate: geometry visual mesh filename=meshes/link16_R.STL
- link R_index_proximal: geometry visual mesh filename=meshes/link15_R.STL
- link R_middle_intermediate: geometry visual mesh filename=meshes/link18_R.STL
- link R_middle_proximal: geometry visual mesh filename=meshes/link17_R.STL
- link R_pinky_intermediate: geometry visual mesh filename=meshes/link22_R.STL
- link R_pinky_proximal: geometry visual mesh filename=meshes/link21_R.STL
- link R_ring_intermediate: geometry visual mesh filename=meshes/link20_R.STL
- link R_ring_proximal: geometry visual mesh filename=meshes/link19_R.STL
- link R_thumb_distal: geometry visual mesh filename=meshes/link14_R.STL
- link R_thumb_intermediate: geometry visual mesh filename=meshes/link13_R.STL
- link R_thumb_proximal: geometry visual mesh filename=meshes/link12_R.STL
- link R_thumb_proximal_base: geometry visual mesh filename=meshes/link11_R.STL
- link left_ankle_pitch_link: geometry visual mesh filename=meshes/left_ankle_pitch_link.STL
- link left_ankle_roll_link: geometry collision cylinder length=0.042 radius=0.005; collision cylinder length=0.076 radius=0.005
- link left_elbow_pitch_link: geometry visual mesh filename=meshes/left_elbow_pitch_link.STL
- link left_elbow_roll_link: geometry visual mesh filename=meshes/left_elbow_roll_link.STL
- link left_hip_pitch_link: geometry visual mesh filename=meshes/left_hip_pitch_link.STL
- link left_hip_roll_link: geometry visual mesh filename=meshes/left_hip_roll_link.STL
- link left_hip_yaw_link: geometry visual mesh filename=meshes/left_hip_yaw_link.STL
- link left_shoulder_pitch_link: geometry visual mesh filename=meshes/left_shoulder_pitch_link.STL
- link left_shoulder_roll_link: geometry visual mesh filename=meshes/left_shoulder_roll_link.STL
- link left_shoulder_yaw_link: geometry visual mesh filename=meshes/left_shoulder_yaw_link.STL
- link left_wrist_pitch_link: geometry visual mesh filename=meshes/left_wrist_pitch_link.STL
- link pelvis: geometry visual mesh filename=meshes/pelvis.STL
- link right_ankle_pitch_link: geometry visual mesh filename=meshes/right_ankle_pitch_link.STL
- link right_ankle_roll_link: geometry collision cylinder length=0.042 radius=0.005; collision cylinder length=0.076 radius=0.005
- link right_elbow_pitch_link: geometry visual mesh filename=meshes/right_elbow_pitch_link.STL
- link right_elbow_roll_link: geometry visual mesh filename=meshes/right_elbow_roll_link.STL
- link right_hip_pitch_link: geometry visual mesh filename=meshes/right_hip_pitch_link.STL
- link right_hip_roll_link: geometry visual mesh filename=meshes/right_hip_roll_link.STL
- link right_hip_yaw_link: geometry visual mesh filename=meshes/right_hip_yaw_link.STL
- link right_shoulder_pitch_link: geometry visual mesh filename=meshes/right_shoulder_pitch_link.STL
- link right_shoulder_roll_link: geometry visual mesh filename=meshes/right_shoulder_roll_link.STL
- link right_shoulder_yaw_link: geometry visual mesh filename=meshes/right_shoulder_yaw_link.STL
- link right_wrist_pitch_link: geometry visual mesh filename=meshes/right_wrist_pitch_link.STL
Joints:
- joint L_index_intermediate_joint: type revolute -> fixed
- joint L_index_proximal_joint: type revolute -> fixed
- joint L_middle_intermediate_joint: type revolute -> fixed
- joint L_middle_proximal_joint: type revolute -> fixed
- joint L_pinky_intermediate_joint: type revolute -> fixed
- joint L_pinky_proximal_joint: type revolute -> fixed
- joint L_ring_intermediate_joint: type revolute -> fixed
- joint L_ring_proximal_joint: type revolute -> fixed
- joint L_thumb_distal_joint: type revolute -> fixed
- joint L_thumb_intermediate_joint: type revolute -> fixed
- joint L_thumb_proximal_pitch_joint: type revolute -> fixed
- joint L_thumb_proximal_yaw_joint: type revolute -> fixed
- joint R_index_intermediate_joint: type revolute -> fixed
- joint R_index_proximal_joint: type revolute -> fixed
- joint R_middle_intermediate_joint: type revolute -> fixed
- joint R_middle_proximal_joint: type revolute -> fixed
- joint R_pinky_intermediate_joint: type revolute -> fixed
- joint R_pinky_proximal_joint: type revolute -> fixed
- joint R_ring_intermediate_joint: type revolute -> fixed
- joint R_ring_proximal_joint: type revolute -> fixed
- joint R_thumb_distal_joint: type revolute -> fixed
- joint R_thumb_intermediate_joint: type revolute -> fixed
- joint R_thumb_proximal_pitch_joint: type revolute -> fixed
- joint R_thumb_proximal_yaw_joint: type revolute -> fixed
- joint left_elbow_pitch_joint: limit lower=-2.53 upper=1.6 effort=18 velocity=20 -> lower=-0.95 upper=3.18 effort=18 velocity=20
- joint left_elbow_roll_joint: limit lower=-2.967 upper=2.967 effort=19 velocity=31.4 -> lower=-3.01 upper=2.75 effort=19 velocity=31.4; type revolute -> fixed
- joint left_shoulder_yaw_joint: limit lower=-3.01 upper=2.66 effort=18 velocity=20 -> lower=-2.66 upper=3.01 effort=18 velocity=20
- joint left_wrist_pitch_joint: limit lower=-0.471 upper=0.349 effort=19 velocity=31.4 -> lower=-0.47 upper=0.47 effort=19 velocity=31.4; type revolute -> fixed
- joint left_wrist_yaw_joint: limit lower=-1.012 upper=1.012 effort=19 velocity=31.4 -> lower=-1.27 upper=1.27 effort=19 velocity=31.4; type revolute -> fixed
- joint right_elbow_pitch_joint: limit lower=-1.6 upper=2.53 effort=18 velocity=20 -> lower=-0.95 upper=3.18 effort=18 velocity=20
- joint right_elbow_roll_joint: limit lower=-2.967 upper=2.967 effort=19 velocity=31.4 -> lower=-2.75 upper=3.01 effort=19 velocity=31.4; type revolute -> fixed
- joint right_shoulder_pitch_joint: limit lower=-1.57 upper=3.14 effort=40 velocity=9 -> lower=-3.14 upper=1.57 effort=40 velocity=9
- joint right_shoulder_yaw_joint: limit lower=-2.66 upper=3.01 effort=18 velocity=20 -> lower=-3.01 upper=2.66 effort=18 velocity=20
- joint right_wrist_pitch_joint: limit lower=-0.471 upper=0.349 effort=19 velocity=31.4 -> lower=-0.47 upper=0.47 effort=19 velocity=31.4; type revolute -> fixed
- joint right_wrist_yaw_joint: limit lower=-1.012 upper=1.012 effort=19 velocity=31.4 -> lower=-1.27 upper=1.27 effort=19 velocity=31.4; type revolute -> fixed
