Commit message: [update] 1. upgrade URDF 2. fix kp/kd bug 3. support new dex3 hand

File: assets/g1/g1_body29_hand14.urdf (robot description, URDF)
Before this commit: robot g1, 50 links, 49 joints
Links:
- removed link imu_link
- removed link left_hand_five_link
- removed link left_hand_four_link
- removed link left_hand_one_link
- removed link left_hand_six_link
- removed link left_hand_three_link
- removed link left_hand_two_link
- removed link left_hand_zero_link
- removed link right_hand_five_link
- removed link right_hand_four_link
- removed link right_hand_one_link
- removed link right_hand_six_link
- removed link right_hand_three_link
- removed link right_hand_two_link
- removed link right_hand_zero_link
- removed link waist_support_link
- added link d435_link
- added link imu_in_pelvis
- added link imu_in_torso
- added link left_hand_index_0_link, mass 0.05885070; collision mesh filename=meshes/left_hand_index_0_link.STL; visual mesh filename=meshes/left_hand_index_0_link.STL
- added link left_hand_index_1_link, mass 0.02030626; collision mesh filename=meshes/left_hand_index_1_link.STL; visual mesh filename=meshes/left_hand_index_1_link.STL
- added link left_hand_middle_0_link, mass 0.05885070; collision mesh filename=meshes/left_hand_middle_0_link.STL; visual mesh filename=meshes/left_hand_middle_0_link.STL
- added link left_hand_middle_1_link, mass 0.02030626; collision mesh filename=meshes/left_hand_middle_1_link.STL; visual mesh filename=meshes/left_hand_middle_1_link.STL
- added link left_hand_thumb_0_link, mass 0.08623657; collision mesh filename=meshes/left_hand_thumb_0_link.STL; visual mesh filename=meshes/left_hand_thumb_0_link.STL
- added link left_hand_thumb_1_link, mass 0.05885070; collision box size=0.02 0.03 0.02; visual mesh filename=meshes/left_hand_thumb_1_link.STL
- added link left_hand_thumb_2_link, mass 0.02030626; collision mesh filename=meshes/left_hand_thumb_2_link.STL; visual mesh filename=meshes/left_hand_thumb_2_link.STL
- added link mid360_link
- added link pelvis_contour_link, mass 0.001; collision mesh filename=meshes/pelvis_contour_link.STL; visual mesh filename=meshes/pelvis_contour_link.STL
- added link right_hand_index_0_link, mass 0.05885070; collision mesh filename=meshes/right_hand_index_0_link.STL; visual mesh filename=meshes/right_hand_index_0_link.STL
- added link right_hand_index_1_link, mass 0.02030626; collision mesh filename=meshes/right_hand_index_1_link.STL; visual mesh filename=meshes/right_hand_index_1_link.STL
- added link right_hand_middle_0_link, mass 0.05885070; collision mesh filename=meshes/right_hand_middle_0_link.STL; visual mesh filename=meshes/right_hand_middle_0_link.STL
- added link right_hand_middle_1_link, mass 0.02030626; collision mesh filename=meshes/right_hand_middle_1_link.STL; visual mesh filename=meshes/right_hand_middle_1_link.STL
- added link right_hand_thumb_0_link, mass 0.08623657; collision mesh filename=meshes/right_hand_thumb_0_link.STL; visual mesh filename=meshes/right_hand_thumb_0_link.STL
- added link right_hand_thumb_1_link, mass 0.05885070; collision box size=0.02 0.03 0.02; visual mesh filename=meshes/right_hand_thumb_1_link.STL
- added link right_hand_thumb_2_link, mass 0.02030626; collision mesh filename=meshes/right_hand_thumb_2_link.STL; visual mesh filename=meshes/right_hand_thumb_2_link.STL
- link left_ankle_roll_link: geometry collision sphere radius=0.005; collision sphere radius=0.005
- link left_shoulder_pitch_link: geometry collision cylinder length=0.05 radius=0.03; visual mesh filename=meshes/left_shoulder_pitch_link.STL
- link left_shoulder_roll_link: geometry collision cylinder length=0.03 radius=0.03; visual mesh filename=meshes/left_shoulder_roll_link.STL
- link logo_link: mass None -> 0.001
- link pelvis: geometry visual mesh filename=meshes/pelvis.STL
- link right_ankle_roll_link: geometry collision sphere radius=0.005; collision sphere radius=0.005
- link right_shoulder_pitch_link: geometry collision cylinder length=0.05 radius=0.03; visual mesh filename=meshes/right_shoulder_pitch_link.STL
- link right_shoulder_roll_link: geometry collision cylinder length=0.03 radius=0.03; visual mesh filename=meshes/right_shoulder_roll_link.STL
- link torso_link: mass 8.562 -> 6.78; geometry collision mesh filename=meshes/torso_link_rev_1_0.STL; visual mesh filename=meshes/torso_link_rev_1_0.STL
- link waist_roll_link: mass 0.047 -> 0.086; geometry visual mesh filename=meshes/waist_roll_link_rev_1_0.STL
- link waist_yaw_link: mass 0.244 -> 0.214; geometry visual mesh filename=meshes/waist_yaw_link_rev_1_0.STL
Joints:
- removed joint imu_joint
- removed joint left_hand_five_joint
- removed joint left_hand_four_joint
- removed joint left_hand_one_joint
- removed joint left_hand_six_joint
- removed joint left_hand_three_joint
- removed joint left_hand_two_joint
- removed joint left_hand_zero_joint
- removed joint right_hand_five_joint
- removed joint right_hand_four_joint
- removed joint right_hand_one_joint
- removed joint right_hand_six_joint
- removed joint right_hand_three_joint
- removed joint right_hand_two_joint
- removed joint right_hand_zero_joint
- removed joint waist_support_joint
- added joint d435_joint: type fixed, parent torso_link, child d435_link, origin xyz=0.0576235 0.01753 0.42987 rpy=0 0.8307767239493009 0
- added joint imu_in_pelvis_joint: type fixed, parent pelvis, child imu_in_pelvis, origin xyz=0.04525 0 -0.08339 rpy=0 0 0
- added joint imu_in_torso_joint: type fixed, parent torso_link, child imu_in_torso, origin xyz=-0.03959 -0.00224 0.14792 rpy=0 0 0
- added joint left_hand_index_0_joint: type revolute, parent left_hand_palm_link, child left_hand_index_0_link, origin xyz=0.0777 0.0016 0.0285 rpy=0 0 0, axis 0 0 1, limit lower=-1.57079632 upper=0 effort=1.4 velocity=12
- added joint left_hand_index_1_joint: type revolute, parent left_hand_index_0_link, child left_hand_index_1_link, origin xyz=0.0458 0 0 rpy=0 0 0, axis 0 0 1, limit lower=-1.74532925 upper=0 effort=1.4 velocity=12
- added joint left_hand_middle_0_joint: type revolute, parent left_hand_palm_link, child left_hand_middle_0_link, origin xyz=0.0777 0.0016 -0.0285 rpy=0 0 0, axis 0 0 1, limit lower=-1.57079632 upper=0 effort=1.4 velocity=12
- added joint left_hand_middle_1_joint: type revolute, parent left_hand_middle_0_link, child left_hand_middle_1_link, origin xyz=0.0458 0 0 rpy=0 0 0, axis 0 0 1, limit lower=-1.74532925 upper=0 effort=1.4 velocity=12
- added joint left_hand_thumb_0_joint: type revolute, parent left_hand_palm_link, child left_hand_thumb_0_link, origin xyz=0.0255 0 0 rpy=0 0 0, axis 0 1 0, limit lower=-1.04719755 upper=1.04719755 effort=2.45 velocity=6.857
- added joint left_hand_thumb_1_joint: type revolute, parent left_hand_thumb_0_link, child left_hand_thumb_1_link, origin xyz=-0.0025 -0.0193 0 rpy=0 0 0, axis 0 0 1, limit lower=-0.72431163 upper=1.04719755 effort=1.4 velocity=12
- added joint left_hand_thumb_2_joint: type revolute, parent left_hand_thumb_1_link, child left_hand_thumb_2_link, origin xyz=0 -0.0458 0 rpy=0 0 0, axis 0 0 1, limit lower=0 upper=1.74532925 effort=1.4 velocity=12
- added joint mid360_joint: type fixed, parent torso_link, child mid360_link, origin xyz=0.0002835 0.00003 0.41618 rpy=0 0.04014257279586953 0
- added joint pelvis_contour_joint: type fixed, parent pelvis, child pelvis_contour_link
- added joint right_hand_index_0_joint: type revolute, parent right_hand_palm_link, child right_hand_index_0_link, origin xyz=0.0777 -0.0016 0.0285 rpy=0 0 0, axis 0 0 1, limit lower=0 upper=1.57079632 effort=1.4 velocity=12
- added joint right_hand_index_1_joint: type revolute, parent right_hand_index_0_link, child right_hand_index_1_link, origin xyz=0.0458 0 0 rpy=0 0 0, axis 0 0 1, limit lower=0 upper=1.74532925 effort=1.4 velocity=12
- added joint right_hand_middle_0_joint: type revolute, parent right_hand_palm_link, child right_hand_middle_0_link, origin xyz=0.0777 -0.0016 -0.0285 rpy=0 0 0, axis 0 0 1, limit lower=0 upper=1.57079632 effort=1.4 velocity=12
- added joint right_hand_middle_1_joint: type revolute, parent right_hand_middle_0_link, child right_hand_middle_1_link, origin xyz=0.0458 0 0 rpy=0 0 0, axis 0 0 1, limit lower=0 upper=1.74532925 effort=1.4 velocity=12
- added joint right_hand_thumb_0_joint: type revolute, parent right_hand_palm_link, child right_hand_thumb_0_link, origin xyz=0.0255 0 0 rpy=0 0 0, axis 0 1 0, limit lower=-1.04719755 upper=1.04719755 effort=2.45 velocity=6.857
- added joint right_hand_thumb_1_joint: type revolute, parent right_hand_thumb_0_link, child right_hand_thumb_1_link, origin xyz=-0.0025 0.0193 0 rpy=0 0 0, axis 0 0 1, limit lower=-1.04719755 upper=0.72431163 effort=1.4 velocity=12
- added joint right_hand_thumb_2_joint: type revolute, parent right_hand_thumb_1_link, child right_hand_thumb_2_link, origin xyz=0 0.0458 0 rpy=0 0 0, axis 0 0 1, limit lower=-1.74532925 upper=0 effort=1.4 velocity=12
- joint head_joint: origin xyz=0.0039635 0 -0.054 rpy=0 0 0 -> xyz=0.0039635 0 -0.044 rpy=0 0 0
- joint left_hip_roll_joint: limit lower=-0.5236 upper=2.9671 effort=88 velocity=32 -> lower=-0.5236 upper=2.9671 effort=139 velocity=20
- joint left_shoulder_pitch_joint: origin xyz=0.0039563 0.10022 0.23778 rpy=0.27931 5.4949E-05 -0.00019159 -> xyz=0.0039563 0.10022 0.24778 rpy=0.27931 5.4949E-05 -0.00019159
- joint logo_joint: origin xyz=0.0039635 0 -0.054 rpy=0 0 0 -> xyz=0.0039635 0 -0.044 rpy=0 0 0
- joint right_hip_roll_joint: limit lower=-2.9671 upper=0.5236 effort=88 velocity=32 -> lower=-2.9671 upper=0.5236 effort=139 velocity=20
- joint right_shoulder_pitch_joint: origin xyz=0.0039563 -0.10021 0.23778 rpy=-0.27931 5.4949E-05 0.00019159 -> xyz=0.0039563 -0.10021 0.24778 rpy=-0.27931 5.4949E-05 0.00019159
- joint waist_pitch_joint: origin xyz=0 0 0.019 rpy=0 0 0 -> xyz=0 0 0 rpy=0 0 0
- joint waist_roll_joint: origin xyz=-0.0039635 0 0.035 rpy=0 0 0 -> xyz=-0.0039635 0 0.044 rpy=0 0 0

File: assets/unitree_hand/unitree_dex3_left.urdf (robot description, URDF)
Before this commit: robot dex3_left, 13 links, 12 joints
Links:
- removed link left_hand_five_link
- removed link left_hand_four_link
- removed link left_hand_one_link
- removed link left_hand_six_link
- removed link left_hand_three_link
- removed link left_hand_two_link
- removed link left_hand_zero_link
- added link base_link_index; visual sphere radius=0.005
- added link base_link_middle; visual sphere radius=0.005
- added link left_hand_index_0_link, mass 0.05885070; collision mesh filename=meshes/left_hand_index_0_link.STL; visual mesh filename=meshes/left_hand_index_0_link.STL
- added link left_hand_index_1_link, mass 0.02030626; collision mesh filename=meshes/left_hand_index_1_link.STL; visual mesh filename=meshes/left_hand_index_1_link.STL
- added link left_hand_middle_0_link, mass 0.05885070; collision mesh filename=meshes/left_hand_middle_0_link.STL; visual mesh filename=meshes/left_hand_middle_0_link.STL
- added link left_hand_middle_1_link, mass 0.02030626; collision mesh filename=meshes/left_hand_middle_1_link.STL; visual mesh filename=meshes/left_hand_middle_1_link.STL
- added link left_hand_thumb_0_link, mass 0.08623657; collision mesh filename=meshes/left_hand_thumb_0_link.STL; visual mesh filename=meshes/left_hand_thumb_0_link.STL
- added link left_hand_thumb_1_link, mass 0.05885070; collision box size=0.02 0.03 0.02; visual mesh filename=meshes/left_hand_thumb_1_link.STL
- added link left_hand_thumb_2_link, mass 0.02030626; collision mesh filename=meshes/left_hand_thumb_2_link.STL; visual mesh filename=meshes/left_hand_thumb_2_link.STL
- link base_link: geometry visual sphere radius=0.01
- link base_link_thumb: geometry visual sphere radius=0.005
Joints:
- removed joint left_hand_five_joint
- removed joint left_hand_four_joint
- removed joint left_hand_one_joint
- removed joint left_hand_six_joint
- removed joint left_hand_three_joint
- removed joint left_hand_two_joint
- removed joint left_hand_zero_joint
- added joint base_index: type fixed, parent base_link, child base_link_index, origin xyz=-0.015 0 0 rpy=0 0 0
- added joint base_middle: type fixed, parent base_link, child base_link_middle, origin xyz=-0.015 0 -0.03 rpy=0 0 0
- added joint left_hand_index_0_joint: type revolute, parent left_hand_palm_link, child left_hand_index_0_link, origin xyz=0.0777 0.0016 0.0285 rpy=0 0 0, axis 0 0 1, limit lower=-1.57079632 upper=0 effort=1.4 velocity=12
- added joint left_hand_index_1_joint: type revolute, parent left_hand_index_0_link, child left_hand_index_1_link, origin xyz=0.0458 0 0 rpy=0 0 0, axis 0 0 1, limit lower=-1.74532925 upper=0 effort=1.4 velocity=12
- added joint left_hand_middle_0_joint: type revolute, parent left_hand_palm_link, child left_hand_middle_0_link, origin xyz=0.0777 0.0016 -0.0285 rpy=0 0 0, axis 0 0 1, limit lower=-1.57079632 upper=0 effort=1.4 velocity=12
- added joint left_hand_middle_1_joint: type revolute, parent left_hand_middle_0_link, child left_hand_middle_1_link, origin xyz=0.0458 0 0 rpy=0 0 0, axis 0 0 1, limit lower=-1.74532925 upper=0 effort=1.4 velocity=12
- added joint left_hand_thumb_0_joint: type revolute, parent left_hand_palm_link, child left_hand_thumb_0_link, origin xyz=0.0255 0 0 rpy=0 0 0, axis 0 1 0, limit lower=-1.04719755 upper=1.04719755 effort=2.45 velocity=6.857
- added joint left_hand_thumb_1_joint: type revolute, parent left_hand_thumb_0_link, child left_hand_thumb_1_link, origin xyz=-0.0025 -0.0193 0 rpy=0 0 0, axis 0 0 1, limit lower=-0.72431163 upper=0.920 effort=1.4 velocity=12
- added joint left_hand_thumb_2_joint: type revolute, parent left_hand_thumb_1_link, child left_hand_thumb_2_link, origin xyz=0 -0.0458 0 rpy=0 0 0, axis 0 0 1, limit lower=0 upper=1.74532925 effort=1.4 velocity=12
- joint base: origin xyz=-0.02 0 0.01 rpy=0 0 -1.57 -> xyz=0 0 0 rpy=0 0 -1.57
- joint base_thumb: child base_link -> base_link_thumb; origin xyz=0.01 0.01 -0.03 rpy=0 0 0 -> xyz=-0.015 0.015 0.02 rpy=0 0 0; parent base_link_thumb -> base_link
- joint index_joint: origin xyz=0.06 -0.003 0 rpy=0 0 0 -> xyz=0.05 0 0 rpy=0 0 0; parent left_hand_six_link -> left_hand_index_1_link
- joint middle_joint: origin xyz=0.06 -0.003 0 rpy=0 0 0 -> xyz=0.05 0 0 rpy=0 0 0; parent left_hand_four_link -> left_hand_middle_1_link
- joint thumb_tip_joint: origin xyz=0.003 -0.06 0 rpy=0 0 0 -> xyz=0 -0.05 0 rpy=0 0 0; parent left_hand_two_link -> left_hand_thumb_2_link

File: assets/unitree_hand/unitree_dex3_right.urdf (robot description, URDF)
Before this commit: robot dex3_right, 13 links, 12 joints
Links:
- removed link right_hand_five_link
- removed link right_hand_four_link
- removed link right_hand_one_link
- removed link right_hand_six_link
- removed link right_hand_three_link
- removed link right_hand_two_link
- removed link right_hand_zero_link
- added link base_link_index; visual sphere radius=0.005
- added link base_link_middle; visual sphere radius=0.005
- added link right_hand_index_0_link, mass 0.05885070; collision mesh filename=meshes/right_hand_index_0_link.STL; visual mesh filename=meshes/right_hand_index_0_link.STL
- added link right_hand_index_1_link, mass 0.02030626; collision mesh filename=meshes/right_hand_index_1_link.STL; visual mesh filename=meshes/right_hand_index_1_link.STL
- added link right_hand_middle_0_link, mass 0.05885070; collision mesh filename=meshes/right_hand_middle_0_link.STL; visual mesh filename=meshes/right_hand_middle_0_link.STL
- added link right_hand_middle_1_link, mass 0.02030626; collision mesh filename=meshes/right_hand_middle_1_link.STL; visual mesh filename=meshes/right_hand_middle_1_link.STL
- added link right_hand_thumb_0_link, mass 0.08623657; collision mesh filename=meshes/right_hand_thumb_0_link.STL; visual mesh filename=meshes/right_hand_thumb_0_link.STL
- added link right_hand_thumb_1_link, mass 0.05885070; collision box size=0.02 0.03 0.02; visual mesh filename=meshes/right_hand_thumb_1_link.STL
- added link right_hand_thumb_2_link, mass 0.02030626; collision mesh filename=meshes/right_hand_thumb_2_link.STL; visual mesh filename=meshes/right_hand_thumb_2_link.STL
- link base_link: geometry visual sphere radius=0.01
- link base_link_thumb: geometry visual sphere radius=0.005
Joints:
- removed joint right_hand_five_joint
- removed joint right_hand_four_joint
- removed joint right_hand_one_joint
- removed joint right_hand_six_joint
- removed joint right_hand_three_joint
- removed joint right_hand_two_joint
- removed joint right_hand_zero_joint
- added joint base_index: type fixed, parent base_link, child base_link_index, origin xyz=-0.015 0 0 rpy=0 0 0
- added joint base_middle: type fixed, parent base_link, child base_link_middle, origin xyz=-0.015 0 0.03 rpy=0 0 0
- added joint right_hand_index_0_joint: type revolute, parent right_hand_palm_link, child right_hand_index_0_link, origin xyz=0.0777 -0.0016 0.0285 rpy=0 0 0, axis 0 0 1, limit lower=0 upper=1.57079632 effort=1.4 velocity=12
- added joint right_hand_index_1_joint: type revolute, parent right_hand_index_0_link, child right_hand_index_1_link, origin xyz=0.0458 0 0 rpy=0 0 0, axis 0 0 1, limit lower=0 upper=1.74532925 effort=1.4 velocity=12
- added joint right_hand_middle_0_joint: type revolute, parent right_hand_palm_link, child right_hand_middle_0_link, origin xyz=0.0777 -0.0016 -0.0285 rpy=0 0 0, axis 0 0 1, limit lower=0 upper=1.57079632 effort=1.4 velocity=12
- added joint right_hand_middle_1_joint: type revolute, parent right_hand_middle_0_link, child right_hand_middle_1_link, origin xyz=0.0458 0 0 rpy=0 0 0, axis 0 0 1, limit lower=0 upper=1.74532925 effort=1.4 velocity=12
- added joint right_hand_thumb_0_joint: type revolute, parent right_hand_palm_link, child right_hand_thumb_0_link, origin xyz=0.0255 0 0 rpy=0 0 0, axis 0 1 0, limit lower=-1.04719755 upper=1.04719755 effort=2.45 velocity=6.857
- added joint right_hand_thumb_1_joint: type revolute, parent right_hand_thumb_0_link, child right_hand_thumb_1_link, origin xyz=-0.0025 0.0193 0 rpy=0 0 0, axis 0 0 1, limit lower=-0.920 upper=0.72431163 effort=1.4 velocity=12
- added joint right_hand_thumb_2_joint: type revolute, parent right_hand_thumb_1_link, child right_hand_thumb_2_link, origin xyz=0 0.0458 0 rpy=0 0 0, axis 0 0 1, limit lower=-1.74532925 upper=0 effort=1.4 velocity=12
- joint base: origin xyz=-0.02 0 0.01 rpy=3.14 0 -1.57 -> xyz=0 0 0 rpy=3.14 0 -1.57
- joint base_thumb: child base_link -> base_link_thumb; origin xyz=0.01 0.01 0.03 rpy=0 0 0 -> xyz=-0.015 0.015 -0.02 rpy=0 0 0; parent base_link_thumb -> base_link
- joint index_joint: origin xyz=0.06 0.003 0 rpy=0 0 0 -> xyz=0.05 0 0 rpy=0 0 0; parent right_hand_six_link -> right_hand_index_1_link
- joint middle_joint: origin xyz=0.06 0.003 0 rpy=0 0 0 -> xyz=0.05 0 0 rpy=0 0 0; parent right_hand_four_link -> right_hand_middle_1_link
- joint thumb_tip_joint: origin xyz=0.003 0.06 0 rpy=0 0 0 -> xyz=0 0.05 0 rpy=0 0 0; parent right_hand_two_link -> right_hand_thumb_2_link
